File: porta_stella.sch (EAGLE design)
At the start: 107 parts, among them CN4 MicroUSB, IC1 74LS00D, J1 2p-smd-1.0-90d, J2 SJ-43516-SMT, SW1 E-SWITCH_JS5208E-SWITCH_JS520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, T1 2N3904, T2 PN3906, T3 PN3906, T4 PN3906, T5 MMUN2133LT1G, U1 TPS61090RSAR, U2 MCP73871, X1 SSW-112-02-G-Q

Commit message: ready for manufacturing
Parts:
- added GOLD_ORB_SM1: OSHWLOGOLOGO5MM, tiny_stella:OSHWLOGOLOGO5MM
- TIA: value ATARI_TIA -> TIA
- renumbered BRIGHT to BRT, R35 to LFT_PADDLE, U$5 to VOL
Changed lines of the file:
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@@
 </classes>
 <parts>
-<part name="TIA" library="tiny_stella" deviceset="ATARI_TIA" device=""/>
+<part name="TIA" library="tiny_stella" deviceset="ATARI_TIA" device="" value="TIA"/>
 <part name="6507" library="tiny_stella" deviceset="MOS_6507" device=""/>
 <part name="6532" library="tiny_stella" deviceset="MOS_6532" device=""/>
@@
 <part name="T1" library="transistor" library_urn="urn:adsk.eagle:library:402" deviceset="*-NPN-" device="SOT23-BEC" package3d_urn="urn:adsk.eagle:package:29919/2" technology="MMBT3904LT1" value="2N3904"/>
 <part name="T2" library="User-Submitted" library_urn="urn:adsk.eagle:library:536" deviceset="TRANSISTOR_PNP" device="PMBT3906" package3d_urn="urn:adsk.eagle:package:40256/1" value="PN3906"/>
-<part name="BRIGHT" library="pot" library_urn="urn:adsk.eagle:library:331" deviceset="TRIM_US-" device="3223G" package3d_urn="urn:adsk.eagle:package:22722/1" value="500k"/>
+<part name="BRT" library="pot" library_urn="urn:adsk.eagle:library:331" deviceset="TRIM_US-" device="3223G" package3d_urn="urn:adsk.eagle:package:22722/1" value="500k"/>
 <part name="R19" library="resistor" library_urn="urn:adsk.eagle:library:348" deviceset="R-US_" device="M0805" package3d_urn="urn:adsk.eagle:package:26079/1" value="1k"/>
 <part name="R20" library="resistor" library_urn="urn:adsk.eagle:library:348" deviceset="R-US_" device="M0805" package3d_urn="urn:adsk.eagle:package:26079/1" value="3.3k"/>
@@
 <part name="CVID" library="wirepad" library_urn="urn:adsk.eagle:library:412" deviceset="WIREPAD" device="2,54/1,1" package3d_urn="urn:adsk.eagle:package:30836/1" value="CVID"/>
 <part name="GND3" library="supply1" library_urn="urn:adsk.eagle:library:371" deviceset="GND" device=""/>
-<part name="R35" library="pot" library_urn="urn:adsk.eagle:library:331" deviceset="TRIM_US-" device="ECP10S" package3d_urn="urn:adsk.eagle:package:22696/1"/>
+<part name="LFT_PADDLE" library="pot" library_urn="urn:adsk.eagle:library:331" deviceset="TRIM_US-" device="ECP10S" package3d_urn="urn:adsk.eagle:package:22696/1"/>
 <part name="GND_A" library="wirepad" library_urn="urn:adsk.eagle:library:412" deviceset="WIREPAD" device="2,54/1,1" package3d_urn="urn:adsk.eagle:package:30836/1" value="GND_A"/>
 <part name="GND_CVID" library="wirepad" library_urn="urn:adsk.eagle:library:412" deviceset="WIREPAD" device="2,54/1,1" package3d_urn="urn:adsk.eagle:package:30836/1" value="GND_CVID"/>
@@
 <part name="J1" library="Seeed-Connector" library_urn="urn:adsk.eagle:library:478" deviceset="SMD-JST-2P-1.0-90D" device="" package3d_urn="urn:adsk.eagle:package:33125/1" value="2p-smd-1.0-90d"/>
 <part name="GND5" library="supply1" library_urn="urn:adsk.eagle:library:371" deviceset="GND" device=""/>
-<part name="U$5" library="tiny_stella" deviceset="3352P-1-103LF" device=""/>
+<part name="VOL" library="tiny_stella" deviceset="3352P-1-103LF" device=""/>
 <part name="GND24" library="supply1" library_urn="urn:adsk.eagle:library:371" deviceset="GND" device=""/>
+<part name="GOLD_ORB_SM1" library="tiny_stella" deviceset="OSHWLOGO" device="LOGO5MM"/>
 </parts>
 <sheets>
@@
 <instance part="T1" gate="G$1" x="254" y="-17.78"/>
 <instance part="T2" gate="G$1" x="266.7" y="-17.78"/>
-<instance part="BRIGHT" gate="G$1" x="236.22" y="-17.78" rot="MR0"/>
+<instance part="BRT" gate="G$1" x="236.22" y="-17.78" rot="MR0"/>
 <instance part="R19" gate="G$1" x="220.98" y="-17.78" rot="MR0"/>
 <instance part="R20" gate="G$1" x="246.38" y="-2.54" rot="MR270"/>
@@
 <instance part="CVID" gate="G$1" x="279.4" y="-25.4" rot="R180"/>
 <instance part="GND3" gate="1" x="228.6" y="30.48" rot="MR0"/>
-<instance part="R35" gate="G$1" x="228.6" y="40.64" rot="R270"/>
+<instance part="LFT_PADDLE" gate="G$1" x="228.6" y="40.64" rot="R270"/>
 <instance part="GND_A" gate="G$1" x="284.48" y="99.06" rot="R270"/>
 <instance part="GND_CVID" gate="G$1" x="284.48" y="-25.4" rot="MR180"/>
@@
 <instance part="J1" gate="G$1" x="-223.52" y="-7.62" rot="MR0"/>
 <instance part="GND5" gate="1" x="284.48" y="86.36" rot="MR0"/>
-<instance part="U$5" gate="G$1" x="172.72" y="12.7" rot="R90"/>
+<instance part="VOL" gate="G$1" x="172.72" y="12.7" rot="R90"/>
 <instance part="GND24" gate="1" x="157.48" y="5.08"/>
+<instance part="GOLD_ORB_SM1" gate="G$1" x="297.18" y="-66.04"/>
 </instances>
 <busses>
@@
 <wire x1="228.6" y1="35.56" x2="228.6" y2="33.02" width="0.1524" layer="91"/>
 <pinref part="GND3" gate="1" pin="GND"/>
-<pinref part="R35" gate="G$1" pin="S"/>
+<pinref part="LFT_PADDLE" gate="G$1" pin="S"/>
 </segment>
 <segment>
@@
 </segment>
 <segment>
-<pinref part="U$5" gate="G$1" pin="E"/>
+<pinref part="VOL" gate="G$1" pin="E"/>
 <wire x1="165.1" y1="12.7" x2="157.48" y2="12.7" width="0.1524" layer="91"/>
 <wire x1="157.48" y1="12.7" x2="157.48" y2="7.62" width="0.1524" layer="91"/>
@@
 <label x="220.98" y="43.18" size="1.778" layer="95" rot="R180"/>
 <wire x1="215.9" y1="40.64" x2="220.98" y2="40.64" width="0.1524" layer="91"/>
-<pinref part="R35" gate="G$1" pin="A"/>
+<pinref part="LFT_PADDLE" gate="G$1" pin="A"/>
 <junction x="215.9" y="40.64"/>
 </segment>
@@
 <pinref part="R21" gate="G$1" pin="1"/>
 <wire x1="246.38" y1="-17.78" x2="246.38" y2="-25.4" width="0.1524" layer="91"/>
-<pinref part="BRIGHT" gate="G$1" pin="A"/>
+<pinref part="BRT" gate="G$1" pin="A"/>
 <wire x1="236.22" y1="-25.4" x2="241.3" y2="-25.4" width="0.1524" layer="91"/>
 <wire x1="241.3" y1="-25.4" x2="241.3" y2="-17.78" width="0.1524" layer="91"/>
@@
 <segment>
 <pinref part="R19" gate="G$1" pin="1"/>
-<pinref part="BRIGHT" gate="G$1" pin="S"/>
+<pinref part="BRT" gate="G$1" pin="S"/>
 <wire x1="226.06" y1="-17.78" x2="231.14" y2="-17.78" width="0.1524" layer="91"/>
 <wire x1="231.14" y1="-25.4" x2="231.14" y2="-17.78" width="0.1524" layer="91"/>
@@
 <wire x1="139.7" y1="35.56" x2="157.48" y2="35.56" width="0.1524" layer="91"/>
 <pinref part="C11" gate="G$1" pin="1"/>
-<pinref part="U$5" gate="G$1" pin="S"/>
+<pinref part="VOL" gate="G$1" pin="S"/>
 <wire x1="172.72" y1="17.78" x2="172.72" y2="22.86" width="0.1524" layer="91"/>
 <wire x1="157.48" y1="35.56" x2="157.48" y2="22.86" width="0.1524" layer="91"/>
@@
 </segment>
 <segment>
-<pinref part="U$5" gate="G$1" pin="A"/>
+<pinref part="VOL" gate="G$1" pin="A"/>
 <wire x1="180.34" y1="12.7" x2="187.96" y2="12.7" width="0.1524" layer="91"/>
 <label x="187.96" y="12.7" size="1.778" layer="95"/>

Commit message: made gerbers and added a to fix list for rev1.1
Parts:
- BRT: value 500k -> 5k
- C11: value 100nF -> 820pF
Connections:
- removed net N$56: SW1.4
- net GND: now also J1.3, J1.4, SW1.COMM.
- net LFT_JOY_DWN: now also SW1.4; no longer SW1.2
- net LFT_JOY_LFT: now also SW1.2; no longer SW1.6
- net LFT_JOY_UP: now also SW1.6; no longer SW1.COMM.
- net N$40: no longer IC1C.I0
- net TIA_RDY: now also IC1C.I0
Other:
- note added: "Control"
